File: EuroCube-65/EuroCube-65.kicad_pcb (KiCad board)
At the start: 2 copper layers, 160 x 100 mm, 105 parts, among them CON1 SERIAL PORT, CON2 PARALLEL PORT, CON3 EXPANSION BUS, IC1 6551A, IC10 GAL16V8, IC11 6522, IC12 6502, IC13 7660, IC2 26LS30, IC3 M3002, IC4 26LS32, IC5 74LS04, IC7 74LS00, IC8 74HCT132, IC9 GAL16V8, T1 BC547, T2 2N7000, T3 2N3906, X1 1.843MHz, X2 32.768kHz, X3 1MHz

Commit message: Updated BOM with correct battery references
Parts:
- B1: value 3V6 -> 2V4-3V6
